Commit message: lift controller changed - effort

File: src/robot_description/urdf/control/ros2_control.xacro (robot description, xacro)
@@ -41,9 +41,9 @@
     </joint>
     <joint name="lift_joint">
-      <!-- ign_ros2_control (Humble): position komutu için P-gain zorunlu -->
-      <param name="position_proportional_gain">50.0</param>
-      <command_interface name="position">
-        <param name="min">${lift_min}</param>
-        <param name="max">${lift_max}</param>
+      <!-- gz_ros2_control Fortress'ta JointVelocityCmd prismatik joint + yerçekimi ile çalışmıyor.
+           effort = lift_mass * g + ekstra = ~20 N tutma, >20 N kaldırma, <20 N indirme -->
+      <command_interface name="effort">
+        <param name="min">-${lift_effort}</param>
+        <param name="max">${lift_effort}</param>
       </command_interface>
       <state_interface name="position"/>

File: src/robot_description/urdf/lift/lift.xacro (robot description, xacro)
@@ -13,5 +13,5 @@
     Platform başlangıç yüksekliği: base_height + lift_z_offset = 0.26 m (LiDAR üstünde)
     Hareket aralığı: 0.0 .. lift_max (0.15 m)
-    Komut: /lift_cmd (std_msgs/Float64) → JointPositionController
+    Çalışan Komut : os2 topic pub - -once /lift_controller/commands std_msgs/msg/Float64MultiArray "data: [-30.0]"
   -->
   <!-- Merkezi direk: en arkada, chassis_link'e sabit -->
@@ -70,5 +70,5 @@
     <limit lower="${lift_min}" upper="${lift_max}"
            effort="${lift_effort}" velocity="${lift_velocity}"/>
-    <dynamics damping="20.0" friction="5.0"/>
+    <dynamics damping="5.0" friction="0.5"/>
   </joint>
 </robot>
