Commit message: slam_nav2 added

File: src/robot_description/urdf/sensors/lidar.xacro (robot description, xacro)
@@ -28,5 +28,5 @@
     <parent link="chassis_link"/>
     <child  link="lidar_link"/>
-    <origin xyz="${base_length/2 - lidar_radius - 0.02} 0 ${base_height + lidar_height/2}"
+    <origin xyz="0 0 ${base_height + lidar_height/2}"
             rpy="0 0 0"/>
   </joint>
